File: kp_towerctrl.kicad_pcb (KiCad board)
At the start: 2 copper layers, 15 parts, among them J1 ext_5v, J2 Conn_02x05_Counter_Clockwise, J3 Conn_02x05_Counter_Clockwise, J4 Conn_02x05_Counter_Clockwise, J5 Conn_02x05_Counter_Clockwise, J6 Conn_02x05_Counter_Clockwise, U1 Teensy4.0, U2 MCP23S17_SP, U3 MCP23S17_SP, U4 MCP3008

Commit message: connect 3.3v
Parts:
- removed J1: ext_5v, Connector_PinHeader_2.54mm:PinHeader_1x02_P2.54mm_Vertical
Connections:
- net 5va renamed 3.3va
- C1 pad 2: 5v -> 3.3v
- C2 pad 2: 5v -> 3.3v
- C3 pad 2: 5v -> 3.3v
- J2 pad 2: 5v -> 3.3v
- J3 pad 2: 5v -> 3.3v
- J4 pad 2: 5v -> 3.3v
- J5 pad 2: 5v -> 3.3v
- NT2 pad 2: 5v -> 3.3v
- U1 pad 1: GND -> gnd
- U1 pad 31: unconnected-(U1-3V3-Pad31) -> 3.3v
- U2 pad 18: 5v -> 3.3v
- U2 pad 9: 5v -> 3.3v
- U3 pad 15: 5v -> 3.3v
- U3 pad 18: 5v -> 3.3v
- U3 pad 9: 5v -> 3.3v
- U4 pad 16: 5v -> 3.3v
